File: _autosave-Minicurso IEEE.sch (KiCad schematic (older format))
At the start: 5 parts

Commit message: Coloquei as footprints la no bixo
Umas cinco, acho
Parts:
- gave numbers to parts that had none: 3
Changed lines of the file:
@@
 $EndComp
 $Comp
-L Device:R_Small R?
+L Device:R_Small R3
 U 1 1 5D4E25C0
 P 3250 4650
-F 0 "R?" H 3309 4696 50  0000 L CNN
+F 0 "R3" H 3309 4696 50  0000 L CNN
 F 1 "10k" H 3309 4605 50  0000 L CNN
 F 2 "" H 3250 4650 50  0001 C CNN
@@
 $EndComp
 $Comp
-L Device:C_Small C?
+L Device:C_Small C1
 U 1 1 5D4E2E2B
 P 2300 4150
-F 0 "C?" V 2071 4150 50  0000 C CNN
+F 0 "C1" V 2071 4150 50  0000 C CNN
 F 1 "20n" V 2162 4150 50  0000 C CNN
 F 2 "" H 2300 4150 50  0001 C CNN
@@
 $EndComp
 $Comp
-L Transistor_BJT:BC548 Q?
+L Transistor_BJT:BC548 Q1
 U 1 1 5D4E34CD
 P 3150 4150
-F 0 "Q?" H 3341 4196 50  0000 L CNN
+F 0 "Q1" H 3341 4196 50  0000 L CNN
 F 1 "BC548" H 3341 4105 50  0000 L CNN
 F 2 "Package_TO_SOT_THT:TO-92_Inline" H 3350 4075 50  0001 L CIN
@@
 $EndComp
 $Comp
-L power:GND #PWR?
+L power:GND #PWR0101
 U 1 1 5D4E5CBC
 P 3250 4900
-F 0 "#PWR?" H 3250 4650 50  0001 C CNN
+F 0 "#PWR0101" H 3250 4650 50  0001 C CNN
 F 1 "GND" H 3255 4727 50  0000 C CNN
 F 2 "" H 3250 4900 50  0001 C CNN
@@
 $EndComp
 $Comp
-L power:VCC #PWR?
+L power:VCC #PWR0102
 U 1 1 5D4E6192
 P 3250 3750
-F 0 "#PWR?" H 3250 3600 50  0001 C CNN
+F 0 "#PWR0102" H 3250 3600 50  0001 C CNN
 F 1 "VCC" H 3267 3923 50  0000 C CNN
 F 2 "" H 3250 3750 50  0001 C CNN
@@
 	3250 4750 3250 4900
 $Comp
-L power:GND #PWR?
+L power:GND #PWR0103
 U 1 1 5D4E6DAC
 P 2850 4900
-F 0 "#PWR?" H 2850 4650 50  0001 C CNN
+F 0 "#PWR0103" H 2850 4650 50  0001 C CNN
 F 1 "GND" H 2855 4727 50  0000 C CNN
 F 2 "" H 2850 4900 50  0001 C CNN
