File: _autosave-Minicurso IEEE.kicad_pcb (KiCad board)
At the start: 2 copper layers, 5 parts, among them Q1 BC548

Commit message: gerbers gerados
Parts:
- C1: value 20n -> 20nF
Routing:
- net Net-(Q1-Pad3): track 0.00 -> 21.1 mm
- net Net-(Q1-Pad2): track 0.00 -> 19.7 mm
- net Net-(C1-Pad1): track 0.00 -> 7.25 mm
- net GND: track 0.00 -> 3.15 mm
Other:
- board outline added: 22.9 x 17.8 mm
Changed lines of the file:
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@@
   (general
     (thickness 1.6)
-    (drawings 0)
-    (tracks 0)
+    (drawings 4)
+    (tracks 18)
     (zones 0)
     (modules 5)
@@
   )
   (setup
-    (last_trace_width 0.25)
+    (last_trace_width 1)
+    (user_trace_width 1)
     (trace_clearance 0.2)
     (zone_clearance 0.508)
@@
       (effects (font (size 1 1) (thickness 0.15)))
     )
-    (fp_text value 20n (at 1.25 2.25) (layer F.Fab)
+    (fp_text value 20nF (at 1.25 2.25) (layer F.Fab)
       (effects (font (size 1 1) (thickness 0.15)))
     )
@@
     )
   )
+  (gr_line (start 53.34 114.3) (end 53.34 96.52) (layer Edge.Cuts) (width 0.05))
+  (gr_line (start 76.2 114.3) (end 53.34 114.3) (layer Edge.Cuts) (width 0.05))
+  (gr_line (start 76.2 96.52) (end 76.2 114.3) (layer Edge.Cuts) (width 0.05))
+  (gr_line (start 53.34 96.52) (end 76.2 96.52) (layer Edge.Cuts) (width 0.05))
+  (segment (start 71.53 105.39) (end 71.53 103.64) (width 1) (layer F.Cu) (net 2))
+  (segment (start 72.580001 106.440001) (end 71.53 105.39) (width 1) (layer F.Cu) (net 2))
+  (segment (start 72.580001 108.670001) (end 72.580001 106.440001) (width 1) (layer F.Cu) (net 2))
+  (segment (start 64.857999 109.660001) (end 71.590001 109.660001) (width 1) (layer F.Cu) (net 2))
+  (segment (start 63.457998 108.26) (end 64.857999 109.660001) (width 1) (layer F.Cu) (net 2))
+  (segment (start 71.590001 109.660001) (end 72.580001 108.670001) (width 1) (layer F.Cu) (net 2))
+  (segment (start 57.91 108.26) (end 63.457998 108.26) (width 1) (layer F.Cu) (net 2))
+  (segment (start 57.91 101.96) (end 57.91 105.11) (width 1) (layer F.Cu) (net 3))
+  (segment (start 70.26 101.89) (end 70.26 103.64) (width 1) (layer F.Cu) (net 3))
+  (segment (start 68.929999 100.559999) (end 70.26 101.89) (width 1) (layer F.Cu) (net 3))
+  (segment (start 62.460001 100.559999) (end 68.929999 100.559999) (width 1) (layer F.Cu) (net 3))
+  (segment (start 57.91 105.11) (end 62.460001 100.559999) (width 1) (layer F.Cu) (net 3))
+  (segment (start 68.58 106.81863) (end 68.58 107.95) (width 1) (layer F.Cu) (net 5))
+  (segment (start 68.58 105.765002) (end 68.58 106.81863) (width 1) (layer F.Cu) (net 5))
+  (segment (start 66.229999 103.415001) (end 68.58 105.765002) (width 1) (layer F.Cu) (net 5))
+  (segment (start 66.229999 102.659999) (end 66.229999 103.415001) (width 1) (layer F.Cu) (net 5))
+  (segment (start 65.53 101.96) (end 66.229999 102.659999) (width 1) (layer F.Cu) (net 5))
+  (segment (start 65.53 105.11) (end 65.53 108.26) (width 1) (layer F.Cu) (net 6))
 )
